File: hardware/drone_fc/drone_fc_v1.0.kicad_sch (KiCad schematic)
At the start: 28 parts, among them J1 Conn_01x05_Pin, J2 Conn_01x08_Socket, J3 Conn_01x03_Pin, SW1 SW_Push, U1 nRF52832-QF48, U2 AMS1117-3.3, Y1 32MHz

Commit message: Added pid, pwm threads
Parts:
- removed AE1: Antenna, RF_Antenna:Johanson_2450AT18x100, symbol Device:Antenna
- removed C11, C12, C13: C, symbol Device:C
- removed C5, C8: 12pF, Capacitor_SMD:C_0603_1608Metric, symbol Device:C
- removed L1: 3.9nH, symbol Device:L
- removed SW1: SW_Push, symbol Switch:SW_Push
- removed U1: nRF52832-QF48, Package_DFN_QFN:QFN-48-1EP_6x6mm_P0.4mm_EP4.6x4.6mm, symbol MCU_Nordic:nRF52832-QFxx
- removed Y1: 32MHz, Crystal:Crystal_SMD_2016-4Pin_2.0x1.6mm, symbol Device:Crystal_GND24
- added CN1: PH2.0 2-pin right-angle SMD connector, easyeda2kicad:CONN-SMD_PH2.0-1X2PW, symbol easyeda2kicad:PH2.0-2P-LT
- added H1, H2, H3, H4: MountingHole, MountingHole:MountingHole_2.2mm_M2, symbol Mechanical:MountingHole
- added R6: 47k, Resistor_SMD:R_0402_1005Metric, symbol Device:R
- added SW1: TS-1187A-B-A-B, easyeda2kicad:SW-SMD_4P-L5.1-W5.1-P3.70-LS6.5-TL_H1.5, symbol easyeda2kicad:TS-1187A-B-A-B
- added U1: E73-2G4M04S1B, easyeda2kicad:WIRELM-SMD_E73-2G4M04S1B, symbol easyeda2kicad:E73-2G4M04S1B
- C1, C6: LCSC Part (none) -> C307331; MPN (none) -> CL05B104KB54PNC; Manufacturer (none) -> Samsung Electro-Mechanics
- C10, C9: LCSC Part (none) -> C361180; MPN (none) -> C2012X5R1A226MT0J0E; Manufacturer (none) -> TDK
- C2: LCSC Part (none) -> C19702; MPN (none) -> CL10A106KP8NNNC; Manufacturer (none) -> Samsung Electro-Mechanics
- C3: value 0.8p -> 100nF; LCSC Part (none) -> C307331; MPN (none) -> CL05B104KB54PNC; Manufacturer (none) -> Samsung Electro-Mechanics
- C4: LCSC Part (none) -> C1546; MPN (none) -> 0402CG101J500NT; Manufacturer (none) -> FH
- C7: LCSC Part (none) -> C52923; MPN (none) -> CL05A105KA5NQNC; Manufacturer (none) -> Samsung Electro-Mechanics
- D1: LCSC Part (none) -> C5372156; MPN (none) -> SML-D13FWT86; Manufacturer (none) -> ROHM Semicon
- J1: value Conn_01x05_Pin -> 1x5 2.54mm male vertical THT header; LCSC Part (none) -> C18213720; MPN (none) -> CS-1109-1X5(L11.5)PA6T; Manufacturer (none) -> CST
- J2: value Conn_01x08_Socket -> 1x8 2.54mm female vertical THT socket; LCSC Part (none) -> C27438; MPN (none) -> 2.54-1*8P母环保; Manufacturer (none) -> BOOMELE
- J3: value Conn_01x03_Pin -> 1x3 2.54mm male vertical THT header; LCSC Part (none) -> C42431683; MPN (none) -> PZ2.54-1X3P-H25; Manufacturer (none) -> JXTCONN
- R1: LCSC Part (none) -> C11702; MPN (none) -> 0402WGF1001TCE; Manufacturer (none) -> UNI-ROYAL
- R2: LCSC Part (none) -> C324831; MPN (none) -> RC-02K1803FT; Manufacturer (none) -> FH
- R3: LCSC Part (none) -> C25741; MPN (none) -> 0402WGF1003TCE; Manufacturer (none) -> UNI-ROYAL
- R4: LCSC Part (none) -> C25744; MPN (none) -> 0402WGF1002TCE; Manufacturer (none) -> UNI-ROYAL
- R5: LCSC Part (none) -> C25900; MPN (none) -> 0402WGF4701TCE; Manufacturer (none) -> UNI-ROYAL
- U2: value AMS1117-3.3 -> TLV1117LV33DCYR; LCSC Part (none) -> C15578; MPN (none) -> TLV1117LV33DCYR; Manufacturer (none) -> Texas Instruments
Connections:
- net 5V is gone; now on net +5V: C9.1, U2.3 (VI)
- net +3V3: now also R5.2, U1.17 (VCC)
- net +VBAT: now also CN1.1
- net BATT_ADC: now also C3.1, U1.9 (P0.28)
- net ESC_PWM: now also R6.1, U1.27 (P0.11)
- net GND: now also C3.2, CN1.2, R6.2, SW1.2 (B), U1.1 (GND), U1.16 (GND), U1.2 (GND), U1.3 (GND), U1.43 (GND), U1.44 (GND); no longer C3.1, R5.2
- net I2C0_SCL: now also U1.29 (P0.13)
- net I2C0_SDA: now also U1.30 (P0.14)
- net MPU6050_INT: now also U1.31 (P0.15)
- net at J1.2 (Pin_2), R4.2: now also SW1.4 (D), U1.37 (P0.21)
- net at J1.3 (Pin_3): now also U1.38 (SWDCLK)
- net at J1.4 (Pin_4): now also U1.39 (SWDIO)
- net at C4.1: now also U1.5 (DEC3)
- net at C6.1: now also U1.15 (DEC1)
- net at C7.1: now also U1.13 (DEC4)
- no-connect marks 31 -> 33
Other:
- moved on the sheet: C1, C2, C4, C6, C7, J1, J2, R2, R3, R4, R5

Commit message: added bluetooth thread, and polished readme
Other:
- note added: "2S LiPo"
- note added: "2S LiPo Input"
- note added: "2S LiPo battery monitor (8.4-6.0 V)"
- note added: "5V BEC from drone ESC"
- note added: "ESC Connector"
- note removed: "2S battery, with ranges from 8.4v - 6.0v"
- note removed: "5v from drone ESC"
- moved on the sheet: C3, CN1, J2, R2, R3, R5
